Commit message: [Fix] Changed mass & inertial matrix
Increased chassis's & wheels' mass to solve the following issue:
 - The robot's front end pops up a bit when it first accelerates, but otherwise appears stable.

File: my_robot/urdf/my_robot.xacro (robot description, xacro)
@@ -15,10 +15,10 @@
     <pose>0 0 0.1 0 0 0</pose>
     <inertial>
-      <mass value="5"/>
+      <mass value="15"/>
       <origin xyz="0 0 0" rpy="0 0 0"/>
       <inertia
-          ixx="0.02808333333" ixy="0" ixz="0"
-          iyy="0.10620833333" iyz="0"
-          izz="0.13020833333"
+          ixx="0.08425" ixy="0" ixz="0"
+          iyy="0.318625" iyz="0"
+          izz="0.390625"
       />
     </inertial>
@@ -51,10 +51,10 @@
   <link name='right_wheel'>
     <inertial>
-      <mass value="0.2"/>
+      <mass value="5"/>
       <origin xyz="0 0 0" rpy="0 1.5707 1.5707" />
       <inertia
-          ixx="0.00052666666" ixy="0" ixz="0"
-          iyy="0.00052666666" iyz="0"
-          izz="0.001"
+          ixx="0.01354166666" ixy="0" ixz="0"
+          iyy="0.01354166666" iyz="0"
+          izz="0.025"
       />
     </inertial>
@@ -62,21 +62,11 @@
       <origin rpy="0 1.5707 1.5707" xyz="0 0 0" />
       <geometry>
-        <cylinder length="0.04" radius="0.1"/>
+        <cylinder length="0.05" radius="0.1"/>
       </geometry>
-      <surface>
-        <friction>
-          <ode>
-            <mu>0</mu>
-            <mu2>0</mu2>
-            <slip1>1.0</slip1>
-            <slip2>1.0</slip2>
-          </ode>
-        </friction>
-      </surface>
     </collision>
     <visual name='right_wheel_visual'>
       <origin rpy="0 1.5707 1.5707" xyz="0 0 0"/>
       <geometry>
-        <cylinder length="0.04" radius="0.1"/>
+        <cylinder length="0.05" radius="0.1"/>
       </geometry>
     </visual>
@@ -95,9 +85,9 @@
     <inertial>
       <origin xyz="0 0 0" rpy="0 1.5707 1.5707" />
-      <mass value="0.2"/>
+      <mass value="5"/>
       <inertia
-          ixx="0.00052666666" ixy="0" ixz="0"
-          iyy="0.00052666666" iyz="0"
-          izz="0.001"
+          ixx="0.01354166666" ixy="0" ixz="0"
+          iyy="0.01354166666" iyz="0"
+          izz="0.025"
       />
     </inertial>
@@ -105,5 +95,5 @@
       <origin xyz="0 0 0" rpy="0 1.5707 1.5707"/>
       <geometry>
-        <cylinder length="0.04" radius="0.1"/>
+        <cylinder length="0.05" radius="0.1"/>
       </geometry>
     </collision>
@@ -111,5 +101,5 @@
       <origin rpy="0 1.5707 1.5707" xyz="0 0 0"/>
       <geometry>
-        <cylinder length="0.04" radius="0.1"/>
+        <cylinder length="0.05" radius="0.1"/>
       </geometry>
     </visual>
